File: USB_Keyboard_32U4/USB_Keyboard_32U4.kicad_pcb (KiCad board)
At the start: 2 copper layers, 38.5 x 37.5 mm, 26 parts, among them J1 USB_C_Receptacle_USB2.0_16P, J2 Conn_02x03_Odd_Even, U1 ATmega32U4-A, Y1 16MHz

Commit message: Update USB-C connector footprint
Replace the USB-C receptacle footprint with the GCT_USB4105-GF-A and update its PCB placement. Refresh the BOM, README, and production outputs to match.
Parts:
- J1: footprint MicroKey_Local:USB4105_JLC_0p20mm_NPTH_Clearance -> Custom Footprints:GCT_USB4105-GF-A
- moved J1 1.08 mm to (116.7, 95.8)
Connections:
- U1 pad 33: HWB -> unconnected-(U1-~{HWB}/PE2-Pad33)
